File: hardware/hv1a/usb-can.brd (EAGLE design)
At the start: 30 x 22 mm, 20 parts, among them CON1 2EDG-4P, Q1 8MHz, U1 CP2130, U2 MCP2515-ML, U3 MCP2562-MF

Commit message: Commit to update
Parts:
- added D2: GREEN, LED:0603
- added D3: RED, LED:0603
- added D4: BLUE, LED:0603
- added R3: 120 Ohms, Resistor:RES0603
- added R4, R5: 330 Ohms, Resistor:RES0603
- C1: value 22pF -> 100nF
- C3: value 100nF -> 22pF
- C4: value 100nF -> 1uF
- C7: value 1uF -> 100nF
- R1: value 120 Ohms -> 10 kOhms
- R2: value 10 kOhms -> 330 Ohms
- U1: value CP2130 -> MCP2515-ML; device Silicon Labs:QFN24 -> Microchip:QFN20
- U2: value MCP2515-ML -> MCP2562-MF; device Microchip:QFN20 -> Microchip:DFN8
- U3: value MCP2562-MF -> CP2130; device Microchip:DFN8 -> Silicon Labs:QFN24
- moved R1 23.2 mm to (6.80, 3.00), turned to 90 degrees
- moved C8 21.4 mm to (5.00, 3.00), turned to 270 degrees
- moved C7 21.0 mm to (19.7, 11.4), turned to 180 degrees
- moved C9 20.6 mm to (9.50, 2.20), turned to 180 degrees
- moved C6 20.2 mm to (3.20, 3.00), turned to 270 degrees
- moved R2 17.2 mm to (11.5, 19.0), turned to 270 degrees
- moved C2 14.3 mm to (22.7, -5.80)
- moved C3 11.7 mm to (11.9, -7.00)
- moved U3 9.69 mm to (13.2, 6.00), turned to 180 degrees
- moved U2 8.51 mm to (19.7, 14.5), turned to 0 degrees
- moved C5 7.11 mm to (8.50, 19.0), turned to 270 degrees
- moved U1 6.60 mm to (19.8, 6.00), turned to 270 degrees
- moved Q1 6.57 mm to (17.9, -8.30)
- moved C4 6.12 mm to (6.70, 19.0), turned to 270 degrees
- moved SJ1 5.81 mm to (23.9, 15.6), flipped to the bottom, turned to 90 degrees
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- renumbered USB2 to USB1
Connections:
- new net CFG_LED: D2.1, U3.12
- new net N$7: D3.2, R4.1
- new net N$8: D4.2, R5.1
- new net N$9: D2.2, R2.1
- new net SPIACT_LED: D4.1, U3.13
- net !CAN_IRQ: now also U1.11, U3.18; no longer U1.18, U2.11
- net !CAN_RST: now also U1.17, U3.21; no longer U1.21, U2.17
- net !CS: now also U1.16, U3.22; no longer U1.22, U2.16
- net 3V3: now also C1.1, C6.1, C7.1, C8.1, R1.2, R4.2, R5.2, U1.18, U2.5, U3.6; no longer C3.1, C4.1, C5.1, C9.1, U1.5, U1.6, U2.18
- net 5V0: now also C4.1, C5.1, U3.7, U3.8; no longer C7.1, C8.1, U1.7, U1.8
- net CANH: now also R3.2, U2.7; no longer R1.2, U3.7
- net CANL: now also U2.6; no longer U3.6
- net CAN_CLK: now also U3.17; no longer U1.17
- net GND: now also D3.1, U1.8, U2.2, U2.9, U3.PAD; no longer U1.2, U2.PAD, U3.8, U3.9
- net MISO: now also U1.15, U3.24; no longer U1.24, U2.15
- net MOSI: now also U1.14, U3.23; no longer U1.23, U2.14
- net N$1: now also C3.1, U1.7; no longer C2.1, U2.7
- net N$2: now also C2.1, U1.6; no longer C1.1, U2.6
- net N$3: now also R3.1; no longer R1.1
- net N$4: now also C9.1, U3.16; no longer C6.1, U1.16
- net N$5: now also R1.1, U3.9; no longer R2.1, U1.9
- net RXCAN: now also U1.20, U2.4; no longer U2.20, U3.4
- net SCK: now also U1.12, U3.1; no longer U1.1, U2.12
- net TXCAN: now also U1.19, U2.1; no longer U2.19, U3.1
- net USB_DM: now also U3.4; no longer U1.4
- net USB_DP: now also U3.3; no longer U1.3
- net VIN: now also U2.3; no longer U3.3
Routing:
- net 3V3: track 0.00 -> 44.0 mm, vias 0 -> 3
- net 5V0: track 0.00 -> 23.8 mm, vias 0 -> 3
- net USB_DP: track 0.00 -> 17.9 mm
- net VIN: track 0.00 -> 17.3 mm, vias 0 -> 1
- net USB_DM: track 0.00 -> 16.2 mm, vias 0 -> 2
- net CANH: track 0.00 -> 10.4 mm
- net CANL: track 0.00 -> 7.67 mm, vias 0 -> 1
- net N$5: track 0.00 -> 6.66 mm
- net N$6: track 0.00 -> 6.35 mm
- net N$4: track 0.00 -> 4.42 mm
- net N$3: track 0.00 -> 2.47 mm, vias 0 -> 1
- net N$9: track 0.00 -> 1.80 mm
- net N$7: track 0.00 -> 1.80 mm
- net N$8: track 0.00 -> 1.80 mm
- added copper zone on layer 1, net GND
- added copper zone on layer 16, net GND
Other:
- outline, holes or cut-outs redrawn

Commit message: Work on PCB
Parts:
- removed C2, C3: 22pF, Capacitor:CAP0603
- removed Q1: 8MHz, Crystal:2-SMD-5X3
- moved C1 0.60 mm to (24.5, 3.00)
Connections:
- removed net N$1: C3.1, Q1.1, U1.7
- removed net N$2: C2.1, Q1.2, U1.6
- net CAN_CLK: now also U1.7
- net GND: no longer C2.2, C3.2
Routing:
- net 3V3: track 44.0 -> 73.8 mm, vias 3 -> 4
- net SPIACT_LED: track 0.00 -> 19.3 mm, vias 0 -> 2
- net CFG_LED: track 0.00 -> 18.6 mm, vias 0 -> 2
- net !CAN_RST: track 0.00 -> 15.5 mm
- net TXCAN: track 0.00 -> 15.5 mm, vias 0 -> 2
- net !CS: track 0.00 -> 13.9 mm
- net MISO: track 0.00 -> 13.8 mm, vias 0 -> 2
- net MOSI: track 0.00 -> 11.0 mm, vias 0 -> 2
- net SCK: track 0.00 -> 10.4 mm, vias 0 -> 2
- net RXCAN: track 0.00 -> 9.21 mm, vias 0 -> 2
- net CAN_CLK: track 0.00 -> 7.57 mm, vias 0 -> 2
- net !CAN_IRQ: track 0.00 -> 6.26 mm, vias 0 -> 2
- net USB_DM: track 16.2 -> 18.0 mm

Commit message: Hardware v1a completed
Parts:
- added LOGO1: IPL-10MM, Silkscreen:IPL_10MM
- added LOGO2: OSHW-LOGOM, Silkscreen:OSHW-LOGO-M
- added SJ2: (no value), Solder Jumper:SJ2C_S
Connections:
- new net N$1: SJ2.2, U2.3
- net 5V0: now also SJ2.3
- net VIN: now also SJ2.1; no longer U2.3
Routing:
- net 5V0: track 23.8 -> 34.9 mm, vias 3 -> 4
- net N$1: track 0.00 -> 6.09 mm, vias 0 -> 1
- net VIN: track 17.3 -> 13.6 mm, vias 1 -> 0
Other:
- board text added: "Designed and assembled in Portugal"
- board text added: "USB-CAN v1a Apr 2019"
