File: hardware/hv1a/usb-can.sch (EAGLE design)
At the start: 5 parts, among them U1 CP2130, U2 MCP2515-ML, U3 MCP2561, U4 MCP1700-330

Commit message: Work
Parts:
- removed U4: MCP1700-330, Microchip:MCP1700-330
- removed USB1: USB_ID_6_SHIELDMICRO_B_SMT, USB Connector:USB_ID_6_SHIELDMICRO_B_SMT
- added C1, C2: 22pF, Capacitor:CAPACITOR-0603
- added C3, C4, C5, C8: 100nF, Capacitor:CAPACITOR-0603
- added C6, C9: 4.7uF, Capacitor:CAPACITOR-0603
- added C7: 1uF, Capacitor:CAPACITOR-0603
- added CON1: 2EDG-4P, Generic Connector:2EDG-4P
- added D1: SP0503BAHT, TVS:SP0503BAHT
- added F1: 500 mA HOLD, PTC Fuses:PTC1206
- added Q1: 8MHz, Crystal:CRYSTAL2-SMD-5X3
- added R1: 120 Ohms, Resistor:RESISTOR-0603
- added R2: 10 kOhms, Resistor:RESISTOR-0603
- added SJ1: (no value), Solder Jumper:SJS
- added USB2: USB_ID_4_SHIELD-MINI-B-SMT, USB Connector:USB_ID_4_SHIELD-MINI-B-SMT
- U3: value MCP2561 -> MCP2562-MF; device Microchip:MCP2561 -> Microchip:MCP2562-MF
Connections:
- new net !CAN_IRQ: U1.GPIO4-!CS4!-EVTCNTR, U2.!INT!
- new net !CAN_RST: U1.GPIO1-!CS1, U2.!RESET!
- new net !CS: U1.GPIO0-!CS0, U2.!CS!
- new net 3V3: C3.C1, C4.C1, C5.C1, C9.C1, R2.2, U1.VDD, U1.VIO, U2.VDD, U3.VIO
- new net 5V0: C7.C1, C8.C1, D1.4, F1.1, U1.VBUS, U1.VREGIN
- new net CANH: CON1-2.S, R1.2, U3.CANH
- new net CANL: CON1-3.S, SJ1.1, U3.CANL
- new net CAN_CLK: U1.GPIO5-!CS5!-CLKOUT
- new net GND: C1.C2, C2.C2, C3.C2, C4.C2, C5.C2, C6.C2, C7.C2, C8.C2, C9.C2, CON1-4.S, D1.1, U1.GND@0, U1.GND@1, U2.VSS, U3.STDBY, U3.VSS, USB2.GND, USB2.SHIELD@0, USB2.SHIELD@1, USB2.SHIELD@2, USB2.SHIELD@3
- new net MISO: U1.MISO, U2.MISO
- new net MOSI: U1.MOSI, U2.MOSI
- new net N$1: C2.C1, Q1.1, U2.OSC1
- new net N$2: C1.C1, Q1.2, U2.OSC2
- new net N$3: R1.1, SJ1.2
- new net N$4: C6.C1, U1.VPP
- new net N$5: R2.1, U1.!RST
- new net N$6: F1.2, USB2.VBUS
- new net RXCAN: U2.RXCAN, U3.RXD
- new net SCK: U1.SCK, U2.SCK
- new net TXCAN: U2.TXCAN, U3.TXD
- new net USB_DM: D1.3, U1.D-, USB2.D-
- new net USB_DP: D1.2, U1.D+, USB2.D+
- new net VIN: CON1-1.S, U3.VDD
Other:
- moved on the sheet: U1, U2, U3

Commit message: Commit to update
Parts:
- added D2: GREEN, LED:LED0603
- added D3: RED, LED:LED0603
- added D4: BLUE, LED:LED0603
- added R3: 120 Ohms, Resistor:RESISTOR-0603
- added R4, R5: 330 Ohms, Resistor:RESISTOR-0603
- C1: value 22pF -> 100nF
- C3: value 100nF -> 22pF
- C4: value 100nF -> 1uF
- C7: value 1uF -> 100nF
- R1: value 120 Ohms -> 10 kOhms
- R2: value 10 kOhms -> 330 Ohms
- U1: value CP2130 -> MCP2515-ML; device Silicon Labs:CP2130 -> Microchip:MCP2515-ML
- U2: value MCP2515-ML -> MCP2562-MF; device Microchip:MCP2515-ML -> Microchip:MCP2562-MF
- U3: value MCP2562-MF -> CP2130; device Microchip:MCP2562-MF -> Silicon Labs:CP2130
- renumbered USB2 to USB1
Connections:
- new net CFG_LED: D2.C, U3.GPIO9-!CS9!-SUSPEND
- new net N$7: D3.A, R4.1
- new net N$8: D4.A, R5.1
- new net N$9: D2.A, R2.1
- new net SPIACT_LED: D4.C, U3.GPIO8-!CS8!-SPIACT
- net !CAN_IRQ: now also U1.!INT!, U3.GPIO4-!CS4!-EVTCNTR; no longer U1.GPIO4-!CS4!-EVTCNTR, U2.!INT!
- net !CAN_RST: now also U1.!RESET!, U3.GPIO1-!CS1; no longer U1.GPIO1-!CS1, U2.!RESET!
- net !CS: now also U1.!CS!, U3.GPIO0-!CS0; no longer U1.GPIO0-!CS0, U2.!CS!
- net 3V3: now also C1.C1, C6.C1, C7.C1, C8.C1, R1.2, R4.2, R5.2, U2.VIO, U3.VDD; no longer C3.C1, C4.C1, C5.C1, C9.C1, U1.VIO, U2.VDD
- net 5V0: now also C4.C1, C5.C1, U3.VBUS, U3.VREGIN; no longer C7.C1, C8.C1, U1.VBUS, U1.VREGIN
- net CANH: now also R3.2, U2.CANH; no longer R1.2, U3.CANH
- net CANL: now also U2.CANL; no longer U3.CANL
- net CAN_CLK: now also U3.GPIO5-!CS5!-CLKOUT; no longer U1.GPIO5-!CS5!-CLKOUT
- net GND: now also D3.C, U1.VSS, U2.STDBY, U3.GND@0, U3.GND@1; no longer U1.GND@0, U1.GND@1, U3.STDBY, U3.VSS
- net MISO: now also U3.MISO; no longer U2.MISO
- net MOSI: now also U3.MOSI; no longer U2.MOSI
- net N$1: now also C3.C1, U1.OSC1; no longer C2.C1, U2.OSC1
- net N$2: now also C2.C1, U1.OSC2; no longer C1.C1, U2.OSC2
- net N$3: now also R3.1; no longer R1.1
- net N$4: now also C9.C1, U3.VPP; no longer C6.C1, U1.VPP
- net N$5: now also R1.1, U3.!RST; no longer R2.1, U1.!RST
- net RXCAN: now also U1.RXCAN, U2.RXD; no longer U2.RXCAN, U3.RXD
- net SCK: now also U3.SCK; no longer U2.SCK
- net TXCAN: now also U1.TXCAN, U2.TXD; no longer U2.TXCAN, U3.TXD
- net USB_DM: now also U3.D-; no longer U1.D-
- net USB_DP: now also U3.D+; no longer U1.D+
- net VIN: now also U2.VDD; no longer U3.VDD
Other:
- moved on the sheet: C1, C2, C3, C4, C5, C6, C7, C8, C9, R1, R2

Commit message: Work on PCB
Parts:
- removed C2, C3: 22pF, Capacitor:CAPACITOR-0603
- removed Q1: 8MHz, Crystal:CRYSTAL2-SMD-5X3
Connections:
- removed net N$1: C3.C1, Q1.1, U1.OSC1
- removed net N$2: C2.C1, Q1.2, U1.OSC2
- net CAN_CLK: now also U1.OSC1
- net GND: no longer C2.C2, C3.C2
Other:
- moved on the sheet: C1
Changed lines of the file:
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@@
 <part name="U1" library="Microchip" deviceset="MCP2515" device="-ML"/>
 <part name="U2" library="Microchip" deviceset="MCP2562" device="-MF"/>
-<part name="Q1" library="Crystal" deviceset="CRYSTAL" device="2-SMD-5X3" value="8MHz"/>
-<part name="C2" library="Capacitor" deviceset="CAPACITOR" device="-0603" value="22pF"/>
-<part name="C3" library="Capacitor" deviceset="CAPACITOR" device="-0603" value="22pF"/>
-<part name="GND7" library="Supply Symbol" deviceset="GND" device=""/>
-<part name="GND8" library="Supply Symbol" deviceset="GND" device=""/>
 <part name="GND9" library="Supply Symbol" deviceset="GND" device=""/>
 <part name="GND4" library="Supply Symbol" deviceset="GND" device=""/>
@@
 <attribute name="VALUE" x="279.4" y="237.49" size="1.27" layer="96"/>
 </instance>
-<instance part="Q1" gate="G$1" x="91.44" y="215.9" smashed="yes" rot="R180">
-<attribute name="NAME" x="88.9" y="214.884" size="1.778" layer="95" rot="R180"/>
-<attribute name="VALUE" x="88.9" y="218.44" size="1.778" layer="96" rot="R180"/>
-</instance>
-<instance part="C2" gate="G$1" x="86.36" y="198.12" smashed="yes" rot="R270">
-<attribute name="VALUE" x="82.0928" y="198.7042" size="1.778" layer="96" ratio="10" rot="SR270"/>
-<attribute name="NAME" x="89.1286" y="199.0344" size="1.778" layer="95" ratio="10" rot="SR270"/>
-</instance>
-<instance part="C3" gate="G$1" x="96.52" y="198.12" smashed="yes" rot="R270">
-<attribute name="VALUE" x="92.2528" y="198.7042" size="1.778" layer="96" ratio="10" rot="SR270"/>
-<attribute name="NAME" x="99.2886" y="199.0344" size="1.778" layer="95" ratio="10" rot="SR270"/>
-</instance>
-<instance part="GND7" gate="G$1" x="86.36" y="185.42" smashed="yes">
-<attribute name="VALUE" x="83.566" y="180.34" size="1.778" layer="96"/>
-</instance>
-<instance part="GND8" gate="G$1" x="96.52" y="185.42" smashed="yes">
-<attribute name="VALUE" x="93.726" y="180.34" size="1.778" layer="96"/>
-</instance>
 <instance part="GND9" gate="G$1" x="119.38" y="185.42" smashed="yes">
 <attribute name="VALUE" x="116.586" y="180.34" size="1.778" layer="96"/>
 </instance>
-<instance part="GND4" gate="G$1" x="73.66" y="185.42" smashed="yes">
-<attribute name="VALUE" x="70.866" y="180.34" size="1.778" layer="96"/>
-</instance>
-<instance part="C1" gate="G$1" x="73.66" y="198.12" smashed="yes" rot="R270">
-<attribute name="VALUE" x="69.3928" y="198.7042" size="1.778" layer="96" ratio="10" rot="SR270"/>
-<attribute name="NAME" x="76.4286" y="199.0344" size="1.778" layer="95" ratio="10" rot="SR270"/>
+<instance part="GND4" gate="G$1" x="93.98" y="185.42" smashed="yes">
+<attribute name="VALUE" x="91.186" y="180.34" size="1.778" layer="96"/>
+</instance>
+<instance part="C1" gate="G$1" x="93.98" y="198.12" smashed="yes" rot="R270">
+<attribute name="VALUE" x="89.7128" y="198.7042" size="1.778" layer="96" ratio="10" rot="SR270"/>
+<attribute name="NAME" x="96.7486" y="199.0344" size="1.778" layer="95" ratio="10" rot="SR270"/>
 </instance>
 <instance part="VIN2" gate="G$1" x="269.24" y="243.84" smashed="yes">
@@
 <attribute name="VALUE" x="261.62" y="160.02" size="1.778" layer="96" rot="R90"/>
 </instance>
-<instance part="3V31" gate="G$1" x="73.66" y="203.2" smashed="yes">
-<attribute name="VALUE" x="71.12" y="200.66" size="1.778" layer="96" rot="R90"/>
+<instance part="3V31" gate="G$1" x="93.98" y="203.2" smashed="yes">
+<attribute name="VALUE" x="91.44" y="200.66" size="1.778" layer="96" rot="R90"/>
 </instance>
 <instance part="3V35" gate="G$1" x="238.76" y="220.98" smashed="yes">
@@
 </busses>
 <nets>
-<net name="N$1" class="0">
-<segment>
-<pinref part="U1" gate="G$1" pin="OSC1"/>
-<wire x1="124.46" y1="218.44" x2="96.52" y2="218.44" width="0.1524" layer="91"/>
-<wire x1="96.52" y1="218.44" x2="96.52" y2="215.9" width="0.1524" layer="91"/>
-<pinref part="C3" gate="G$1" pin="C1"/>
-<pinref part="Q1" gate="G$1" pin="1"/>
-<wire x1="96.52" y1="215.9" x2="96.52" y2="198.12" width="0.1524" layer="91"/>
-<wire x1="93.98" y1="215.9" x2="96.52" y2="215.9" width="0.1524" layer="91"/>
-<junction x="96.52" y="215.9"/>
-</segment>
-</net>
-<net name="N$2" class="0">
-<segment>
-<pinref part="U1" gate="G$1" pin="OSC2"/>
-<wire x1="124.46" y1="220.98" x2="86.36" y2="220.98" width="0.1524" layer="91"/>
-<pinref part="C2" gate="G$1" pin="C1"/>
-<wire x1="86.36" y1="198.12" x2="86.36" y2="215.9" width="0.1524" layer="91"/>
-<pinref part="Q1" gate="G$1" pin="2"/>
-<wire x1="86.36" y1="215.9" x2="86.36" y2="220.98" width="0.1524" layer="91"/>
-<wire x1="88.9" y1="215.9" x2="86.36" y2="215.9" width="0.1524" layer="91"/>
-<junction x="86.36" y="215.9"/>
-</segment>
-</net>
 <net name="GND" class="0">
-<segment>
-<pinref part="GND8" gate="G$1" pin="GND"/>
-<pinref part="C3" gate="G$1" pin="C2"/>
-<wire x1="96.52" y1="185.42" x2="96.52" y2="190.5" width="0.1524" layer="91"/>
-</segment>
-<segment>
-<pinref part="GND7" gate="G$1" pin="GND"/>
-<pinref part="C2" gate="G$1" pin="C2"/>
-<wire x1="86.36" y1="185.42" x2="86.36" y2="190.5" width="0.1524" layer="91"/>
-</segment>
 <segment>
 <pinref part="GND9" gate="G$1" pin="GND"/>
@@
 <pinref part="C1" gate="G$1" pin="C2"/>
 <pinref part="GND4" gate="G$1" pin="GND"/>
-<wire x1="73.66" y1="190.5" x2="73.66" y2="185.42" width="0.1524" layer="91"/>
+<wire x1="93.98" y1="190.5" x2="93.98" y2="185.42" width="0.1524" layer="91"/>
 </segment>
 <segment>
@@
 <pinref part="C1" gate="G$1" pin="C1"/>
 <pinref part="3V31" gate="G$1" pin="3V3"/>
-<wire x1="73.66" y1="198.12" x2="73.66" y2="203.2" width="0.1524" layer="91"/>
+<wire x1="93.98" y1="198.12" x2="93.98" y2="203.2" width="0.1524" layer="91"/>
 </segment>
 <segment>
@@
 <label x="342.9" y="124.46" size="1.778" layer="95" xref="yes"/>
 </segment>
-</net>
+<segment>
+<pinref part="U1" gate="G$1" pin="OSC1"/>
+<wire x1="124.46" y1="218.44" x2="119.38" y2="218.44" width="0.1524" layer="91"/>
+<label x="119.38" y="218.44" size="1.778" layer="95" rot="R180" xref="yes"/>
+</segment>
+</net>

Commit message: Hardware v1a completed
Parts:
- added LOGO1: IPL-10MM, Silkscreen:IPL-10MM
- added LOGO2: OSHW-LOGOM, Silkscreen:OSHW-LOGOM
- added SJ2: (no value), Solder Jumper:SJ2CS
Connections:
- new net N$1: SJ2.2, U2.VDD
- net 5V0: now also SJ2.3
- net VIN: now also SJ2.1; no longer U2.VDD
Changed lines of the file:
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@@
 <part name="R2" library="Resistor" deviceset="RESISTOR" device="-0603" value="330 Ohms"/>
 <part name="3V39" library="Supply Symbol" deviceset="3V3" device=""/>
+<part name="LOGO1" library="Silkscreen" deviceset="IPL" device="-10MM"/>
+<part name="LOGO2" library="Silkscreen" deviceset="OSHW-LOGO" device="M"/>
+<part name="SJ2" library="Solder Jumper" deviceset="SJ2C" device="S"/>
+<part name="5V03" library="Supply Symbol" deviceset="5V0" device=""/>
 </parts>
 <sheets>
@@
 <attribute name="NAME" x="96.7486" y="199.0344" size="1.778" layer="95" ratio="10" rot="SR270"/>
 </instance>
-<instance part="VIN2" gate="G$1" x="269.24" y="243.84" smashed="yes">
-<attribute name="VALUE" x="266.7" y="241.3" size="1.778" layer="96" rot="R90"/>
+<instance part="VIN2" gate="G$1" x="261.62" y="246.38" smashed="yes">
+<attribute name="VALUE" x="259.08" y="243.84" size="1.778" layer="96" rot="R90"/>
 </instance>
 <instance part="GND17" gate="G$1" x="269.24" y="203.2" smashed="yes">
@@
 <attribute name="VALUE" x="236.22" y="218.44" size="1.778" layer="96" rot="R90"/>
 </instance>
-<instance part="3V37" gate="G$1" x="261.62" y="243.84" smashed="yes">
-<attribute name="VALUE" x="259.08" y="241.3" size="1.778" layer="96" rot="R90"/>
+<instance part="3V37" gate="G$1" x="251.46" y="246.38" smashed="yes">
+<attribute name="VALUE" x="248.92" y="243.84" size="1.778" layer="96" rot="R90"/>
 </instance>
 <instance part="3V32" gate="G$1" x="119.38" y="241.3" smashed="yes">
@@
 <instance part="3V39" gate="G$1" x="307.34" y="76.2" smashed="yes">
 <attribute name="VALUE" x="304.8" y="73.66" size="1.778" layer="96" rot="R90"/>
+</instance>
+<instance part="LOGO1" gate="G$1" x="368.3" y="27.94" smashed="yes"/>
+<instance part="LOGO2" gate="G$1" x="269.24" y="17.78" smashed="yes"/>
+<instance part="SJ2" gate="G$1" x="269.24" y="241.3" smashed="yes" rot="R90">
+<attribute name="NAME" x="268.859" y="243.84" size="1.778" layer="95" rot="R90"/>
+<attribute name="VALUE" x="271.145" y="243.84" size="1.778" layer="96" rot="R90"/>
+</instance>
+<instance part="5V03" gate="G$1" x="276.86" y="246.38" smashed="yes">
+<attribute name="VALUE" x="274.32" y="243.84" size="1.778" layer="96" rot="R90"/>
 </instance>
 </instances>
@@
 <net name="VIN" class="0">
 <segment>
-<pinref part="U2" gate="G$1" pin="VDD"/>
-<pinref part="VIN2" gate="G$1" pin="VIN"/>
-<wire x1="274.32" y1="233.68" x2="269.24" y2="233.68" width="0.1524" layer="91"/>
-<wire x1="269.24" y1="233.68" x2="269.24" y2="243.84" width="0.1524" layer="91"/>
-</segment>
-<segment>
 <pinref part="CON1" gate="-1" pin="S"/>
 <pinref part="VIN1" gate="G$1" pin="VIN"/>
 <wire x1="83.82" y1="147.32" x2="76.2" y2="147.32" width="0.1524" layer="91"/>
 <wire x1="76.2" y1="147.32" x2="76.2" y2="154.94" width="0.1524" layer="91"/>
+</segment>
+<segment>
+<pinref part="SJ2" gate="G$1" pin="1"/>
+<pinref part="VIN2" gate="G$1" pin="VIN"/>
+<wire x1="264.16" y1="241.3" x2="261.62" y2="241.3" width="0.1524" layer="91"/>
+<wire x1="261.62" y1="241.3" x2="261.62" y2="246.38" width="0.1524" layer="91"/>
 </segment>
 </net>
@@
 <junction x="86.36" y="88.9"/>
 </segment>
+<segment>
+<pinref part="SJ2" gate="G$1" pin="3"/>
+<pinref part="5V03" gate="G$1" pin="5V0"/>
+<wire x1="274.32" y1="241.3" x2="276.86" y2="241.3" width="0.1524" layer="91"/>
+<wire x1="276.86" y1="241.3" x2="276.86" y2="246.38" width="0.1524" layer="91"/>
+</segment>
 </net>
 <net name="3V3" class="0">
@@
 <segment>
 <pinref part="U2" gate="G$1" pin="VIO"/>
-<wire x1="274.32" y1="231.14" x2="261.62" y2="231.14" width="0.1524" layer="91"/>
-<wire x1="261.62" y1="231.14" x2="261.62" y2="243.84" width="0.1524" layer="91"/>
+<wire x1="274.32" y1="231.14" x2="251.46" y2="231.14" width="0.1524" layer="91"/>
+<wire x1="251.46" y1="231.14" x2="251.46" y2="246.38" width="0.1524" layer="91"/>
 <pinref part="3V37" gate="G$1" pin="3V3"/>
 </segment>
@@
 </segment>
 </net>
+<net name="N$1" class="0">
+<segment>
+<pinref part="U2" gate="G$1" pin="VDD"/>
+<wire x1="274.32" y1="233.68" x2="269.24" y2="233.68" width="0.1524" layer="91"/>
+<pinref part="SJ2" gate="G$1" pin="2"/>
+<wire x1="269.24" y1="236.22" x2="269.24" y2="233.68" width="0.1524" layer="91"/>
+</segment>
+</net>
 </nets>
 </sheet>
@@
 </drawing>
 <compatibility>
+<note version="6.3" minversion="6.2.2" severity="warning">
+Since Version 6.2.2 text objects can contain more than one line,
+which will not be processed correctly with this version.
+</note>
 <note version="8.3" severity="warning">
 Since Version 8.3, EAGLE supports URNs for individual library
